Commit message: training ole sophie

File: xarm-gym-env-pybullet/env/xarm7_pd.urdf (robot description, URDF)
Before this commit: robot xarm7_with_gripper, 14 links, 13 joints
Links:
- link link_base: mass 0.88556 -> 0
- link panda_hand: mass .81 -> 0
- link panda_leftfinger: mass 0.1 -> 0; geometry collision box size=0 0 0; visual mesh filename=meshes/visual/finger.obj
- link panda_rightfinger: mass 0.1 -> 0; geometry collision box size=0 0 0; visual mesh filename=meshes/visual/finger.obj
